File: Schematic-PCB/Ball-20240325/Ball-20240325.kicad_sch (KiCad schematic)
At the start: 0 parts

Commit message: コートの3Dモデルの追加+回路図編集
Parts:
- added C1, C10, C11, C12, C13, C14, C15, C16, C2, C3, C4, C5, C6, C7, C8, C9: 0.33uF, symbol Device:C_Small
- added R1, R10, R11, R12, R13, R14, R15, R16, R2, R3, R4, R5, R6, R7, R8, R9: 39K, symbol Device:R_Small
- added U1, U10, U11, U12, U13, U14, U15, U16, U2, U3, U4, U5, U6, U7, U8, U9: TSSP58P38, OptoDevice:Vishay_MINICAST-3Pin, symbol Sensor_Proximity:TSSP58P38
Connections:
- new net: R6.1, U6.1 (OUT)
- new net: R3.1, U3.1 (OUT)
- new net: R10.1, U10.1 (OUT)
- new net: R4.1, U4.1 (OUT)
- new net: R12.1, U12.1 (OUT)
- new net: R1.1, U1.1 (OUT)
- new net: R8.1, U8.1 (OUT)
- new net: R11.1, U11.1 (OUT)
- new net: R15.1, U15.1 (OUT)
- new net: R13.1, U13.1 (OUT)
- new net: R5.1, U5.1 (OUT)
- new net: R14.1, U14.1 (OUT)
- new net: R7.1, U7.1 (OUT)
- new net: R16.1, U16.1 (OUT)
- new net: R9.1, U9.1 (OUT)
- new net: R2.1, U2.1 (OUT)
- new net GND: C1.2, C10.2, C11.2, C12.2, C13.2, C14.2, C15.2, C16.2, C2.2, C3.2, C4.2, C5.2, C6.2, C7.2, C8.2, C9.2, U1.2 (GND), U10.2 (GND), U11.2 (GND), U12.2 (GND), U13.2 (GND), U14.2 (GND), U15.2 (GND), U16.2 (GND), U2.2 (GND), U3.2 (GND), U4.2 (GND), U5.2 (GND), U6.2 (GND), U7.2 (GND), U8.2 (GND), U9.2 (GND)
- new net VCC: U1.3 (Vs), U10.3 (Vs), U11.3 (Vs), U12.3 (Vs), U13.3 (Vs), U14.3 (Vs), U15.3 (Vs), U16.3 (Vs), U2.3 (Vs), U3.3 (Vs), U4.3 (Vs), U5.3 (Vs), U6.3 (Vs), U7.3 (Vs), U8.3 (Vs), U9.3 (Vs)
- new net ball01: C1.1, R1.2
- new net ball02: C2.1, R2.2
- new net ball03: C3.1, R3.2
- new net ball04: C4.1, R4.2
- new net ball05: C5.1, R5.2
- new net ball06: C6.1, R6.2
- new net ball07: C7.1, R7.2
- new net ball08: C8.1, R8.2
- new net ball09: C9.1, R9.2
- new net ball10: C10.1, R10.2
- new net ball11: C11.1, R11.2
- new net ball12: C12.1, R12.2
- new net ball13: C13.1, R13.2
- new net ball14: C14.1, R14.2
- new net ball15: C15.1, R15.2
- new net ball16: C16.1, R16.2
Other:
- note added: "CPU"
- note added: "Sensor"
