File: Schematic-PCB/(練習用) ATmega2560/ATmega2560.kicad_pcb (KiCad board)
At the start: 0 parts

Commit message: (練習用)ATMega2560のPCBを編集
Parts:
- added BZ1: Buzzer, @MyLibrary:PKM13EPYH4000-A0, F.Cu at (78.2, 57.4)
- added C1: C, Capacitor_SMD:C_0805_2012Metric, F.Cu at (52.1, 30.5)
- added D1: LED, LED_SMD:LED_0603_1608Metric, F.Cu at (76.6, 83.3)
- added D2: LED, LED_SMD:LED_0603_1608Metric, F.Cu at (79.6, 83.3)
- added D3: LED, LED_SMD:LED_0603_1608Metric, F.Cu at (82.5, 83.3)
- added J1: Conn_01x20_Pin, Connector_IDC:IDC-Header_2x10_P2.54mm_Vertical, F.Cu at (71.9, 27.6)
- added J2: Conn_01x06_Pin, Connector_JST:JST_XH_B6B-XH-A_1x06_P2.50mm_Vertical, B.Cu at (53.3, 54.8)
- added J3: Conn_01x06_Pin, Connector_JST:JST_XH_B6B-XH-A_1x06_P2.50mm_Vertical, B.Cu at (115.6, 67.3)
- added J4: Conn_01x26_Pin, Connector_IDC:IDC-Header_2x13_P2.54mm_Vertical, B.Cu at (68.6, 41.9)
- added J5: Conn_01x04_Socket, Connector_PinSocket_2.54mm:PinSocket_1x04_P2.54mm_Vertical, B.Cu at (114.3, 40.6)
- added J6: Conn_01x02_Pin, Connector_JST:JST_XH_S2B-XH-A-1_1x02_P2.50mm_Horizontal, F.Cu at (62.5, 29.5)
- added J7: Conn_01x03_Pin, Connector_JST:JST_XH_S3B-XH-A-1_1x03_P2.50mm_Horizontal, B.Cu at (56.5, 44.4)
- added JP1: Jumper_2_Open, Jumper:SolderJumper-2_P1.3mm_Open_Pad1.0x1.5mm, F.Cu at (54.4, 83.8)
- added JP2: Jumper_2_Open, Jumper:SolderJumper-2_P1.3mm_Open_Pad1.0x1.5mm, F.Cu at (57.9, 83.8)
- added JP3: Jumper_2_Open, Jumper:SolderJumper-2_P1.3mm_Open_Pad1.0x1.5mm, F.Cu at (61.5, 83.8)
- added JP4: Jumper_2_Open, Jumper:SolderJumper-2_P1.3mm_Open_Pad1.0x1.5mm, F.Cu at (65.0, 83.8)
- added JP5: Jumper_2_Open, Jumper:SolderJumper-2_P1.3mm_Open_Pad1.0x1.5mm, F.Cu at (68.6, 83.8)
- added R1: 1K, Resistor_SMD:R_0805_2012Metric, F.Cu at (96.5, 74.9)
- added R10: 330, Resistor_SMD:R_0805_2012Metric, F.Cu at (79.6, 79.5)
- added R11: 330, Resistor_SMD:R_0805_2012Metric, F.Cu at (82.5, 79.5)
- added R12: 1K, Resistor_SMD:R_0805_2012Metric, F.Cu at (115.6, 74.9)
- added R13: 10K, Resistor_SMD:R_0805_2012Metric, F.Cu at (118.1, 74.9)
- added R14: 1K, Resistor_SMD:R_0805_2012Metric, F.Cu at (57.3, 49.0)
- added R2: 10K, Resistor_SMD:R_0805_2012Metric, F.Cu at (99.1, 74.9)
- added R3: 1K, Resistor_SMD:R_0805_2012Metric, F.Cu at (102.9, 74.9)
- added R4: 10K, Resistor_SMD:R_0805_2012Metric, F.Cu at (105.4, 74.9)
- added R5: 1K, Resistor_SMD:R_0805_2012Metric, F.Cu at (109.2, 74.9)
- added R6: 10K, Resistor_SMD:R_0805_2012Metric, F.Cu at (111.8, 74.9)
- added R7: 1K, Resistor_SMD:R_0805_2012Metric, F.Cu at (87.2, 73.3)
- added R8: 10K, Resistor_SMD:R_0805_2012Metric, F.Cu at (90.2, 73.3)
- added R9: 330, Resistor_SMD:R_0805_2012Metric, F.Cu at (76.7, 79.5)
- added SW1: SW_Push, @MyLibrary:TVBP06-BN043CB-B, F.Cu at (96.5, 81.3)
- added SW2: SW_Push, @MyLibrary:TVBP06-BN043CB-B, F.Cu at (102.9, 81.3)
- added SW3: SW_Push, @MyLibrary:TVBP06-BN043CB-B, F.Cu at (109.2, 81.3)
- added SW4: SW_Push, @MyLibrary:TVBP06-BN043CB-B, F.Cu at (115.6, 81.3)
- added SW6: SW_SPDT, @MyLibrary:SS12D01G4-G_2, F.Cu at (88.9, 80.0)
- added U1: MEGA_PRO_EMBED_CH340G___ATMEGA2560, ATMega2560:ATMega2560, F.Cu at (84.3, 50.8)
- added U2: ~, @MyLibrary:BNO055, F.Cu at (95.3, 57.1)
- added U3: ~, Connector_IDC:IDC-Header_2x05_P2.54mm_Vertical, F.Cu at (55.9, 77.5)
Routing:
- net MD2_EN1: track 0.00 -> 46.6 mm
- net MD2_EN2: track 0.00 -> 46.4 mm
- net MD1_PH1: track 0.00 -> 37.8 mm
- net SDA: track 0.00 -> 36.9 mm
- net KICKER: track 0.00 -> 36.8 mm
- net MD2_PH2: track 0.00 -> 32.0 mm
- net SCL: track 0.00 -> 32.0 mm
- net MD2_PH1: track 0.00 -> 30.7 mm
- net LS_07: track 0.00 -> 29.0 mm
- net LS_13: track 0.00 -> 28.6 mm
- net LS_01: track 0.00 -> 28.3 mm
- net LS_11: track 0.00 -> 28.2 mm
- net LS_09: track 0.00 -> 28.2 mm
- net LS_05: track 0.00 -> 28.2 mm
- net LS_03: track 0.00 -> 28.2 mm
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Other:
- copper layers 0 -> 2
