File: Schematic-PCB/UI-20240325/UI-20240325.kicad_pcb (KiCad board)
At the start: 0 parts

Commit message: UI基板のPCBデザインを作成
決定ボタンのみフットプリントが決定しておらず未完成
Parts:
- added A: SW_SPDT, @2024-UI:2MS1-T1-B4-VS2-Q-E-S, F.Cu at (111.5, 96.6)
- added B: SW_SPDT, @2024-UI:2MS1-T1-B4-VS2-Q-E-S, F.Cu at (111.5, 80.6)
- added BZ1: Buzzer, @2024-UI:PKM13EPYH4000-A0, B.Cu at (78.0, 87.0)
- added J1: Conn_01x10_Pin, Connector_JST:JST_XH_B10B-XH-A_1x10_P2.50mm_Vertical, F.Cu at (101.5, 61.2)
- added R1: 1K, Resistor_SMD:R_0603_1608Metric, B.Cu at (108.0, 79.8)
- added R10: 10K, Resistor_SMD:R_0603_1608Metric, B.Cu at (101.2, 101.5)
- added R2: 1K, Resistor_SMD:R_0603_1608Metric, B.Cu at (108.0, 95.8)
- added R3: 10K, Resistor_SMD:R_0603_1608Metric, B.Cu at (106.0, 79.8)
- added R4: 10K, Resistor_SMD:R_0603_1608Metric, B.Cu at (106.0, 95.8)
- added R5: 1K, Resistor_SMD:R_0603_1608Metric, B.Cu at (99.2, 74.8)
- added R6: 1K, Resistor_SMD:R_0603_1608Metric, B.Cu at (105.7, 123.1)
- added R7: 1K, Resistor_SMD:R_0603_1608Metric, B.Cu at (99.2, 99.8)
- added R8: 10K, Resistor_SMD:R_0603_1608Metric, B.Cu at (101.2, 76.5)
- added R9: 10K, Resistor_SMD:R_0603_1608Metric, B.Cu at (100.7, 123.6)
- added REF**: MountingHole_3.2mm_M3, MountingHole:MountingHole_3.2mm_M3, F.Cu at (59.4, 88.1)
- added REF**: MountingHole_3.2mm_M3, MountingHole:MountingHole_3.2mm_M3, F.Cu at (121.1, 88.1)
- added REF**: MountingHole_3.2mm_M3, MountingHole:MountingHole_3.2mm_M3, F.Cu at (52.0, 80.0)
- added REF**: MountingHole_3.2mm_M3, MountingHole:MountingHole_3.2mm_M3, F.Cu at (128.5, 80.0)
- added U1: ~, @2024-UI:Display, F.Cu at (78.0, 76.0)
- added ▲: SW_Push, @2024-UI:TVBP06-B043C, F.Cu at (100.2, 75.6)
- added ▼: SW_Push, @2024-UI:TVBP06-B043C, F.Cu at (100.2, 100.6)
Routing:
- net +3.3V: track 0.00 -> 78.2 mm
- net SW-TAC-3: track 0.00 -> 43.1 mm
- net SW-TOG-2: track 0.00 -> 39.6 mm
- net BUZZER: track 0.00 -> 27.3 mm
- net SW-TOG-1: track 0.00 -> 22.6 mm
- net SW-TAC-1: track 0.00 -> 16.0 mm
- net SCL: track 0.00 -> 15.7 mm
- net SDA: track 0.00 -> 15.7 mm
- net Net-(SW2-B): track 0.00 -> 5.50 mm
- net Net-(R5-Pad2): track 0.00 -> 4.25 mm
- net Net-(R10-Pad2): track 0.00 -> 4.25 mm
- added copper zone on B.Cu, net GND
- added copper zone on F.Cu, net GND
Other:
- board outline added: 82.9 x 53.9 mm
- copper layers 0 -> 2
