File: Schematic-PCB/UI-20240325/UI-20240325.kicad_pcb (KiCad board)
At the start: 2 copper layers, 65.5 x 30.7 mm, 22 parts, among them J1 Conn, SW1 SW_SPDT, SW2 SW_Push, SW3 SW_Push, SW4 SW_Push, SW5 SW_Push

Commit message: update: UI基板のボタンの1つが+3.3Vに接続されていなかったのを修正した
Routing:
- net +3.3V: track 123.7 -> 128.1 mm
- net unconnected-(SW1-C-Pad3): track 0.00 -> 0.98 mm
Other:
- board text added: "UI-Board #004"
- board text removed: "UI-Board #003"

Commit message: UI基板の各ボタンにチャタリング防止用コンデンサを配置した
ただしトグルスイッチを除く()
Parts:
- added C1: 0.1uF, Capacitor_SMD:C_0603_1608Metric, B.Cu at (-19.5, 27.0)
- added C2: 0.1uF, Capacitor_SMD:C_0603_1608Metric, B.Cu at (19.5, 13.0)
- added C3: 0.1uF, Capacitor_SMD:C_0603_1608Metric, B.Cu at (19.5, 20.0)
- added C4: 0.1uF, Capacitor_SMD:C_0603_1608Metric, B.Cu at (19.5, 27.0)
Connections:
- J1 pad 3: SW-TAC-1 -> SW-TOG
- J1 pad 4: SW-TAC-2 -> SW-TAC-1
- J1 pad 5: SW-TAC-3 -> SW-TAC-2
- J1 pad 6: SW-TAC-4 -> SW-TAC-3
- J1 pad 7: SW-TAC-5 -> SW-TAC-4
- R1 pad 1: SW-TAC-1 -> SW-TOG
- R3 pad 1: SW-TAC-2 -> SW-TAC-1
- R5 pad 1: SW-TAC-3 -> SW-TAC-2
- R7 pad 1: SW-TAC-4 -> SW-TAC-3
- R9 pad 1: SW-TAC-5 -> SW-TAC-4
Routing:
- net SW-TAC-5: track 29.6 -> 0.00 mm
- net SW-TOG: track 0.00 -> 27.4 mm
- net +3.3V: track 128.1 -> 144.3 mm
- net SW-TAC-2: track 35.1 -> 20.7 mm
- net SW-TAC-1: track 27.4 -> 35.1 mm
- net SW-TAC-4: track 24.2 -> 29.6 mm
- net Net-(C4-Pad1): track 5.18 -> 9.18 mm
- net Net-(C3-Pad1): track 5.18 -> 9.18 mm
- net Net-(C1-Pad1): track 5.18 -> 9.18 mm
- net Net-(C2-Pad1): track 5.18 -> 9.18 mm
- net SW-TAC-3: track 20.7 -> 24.2 mm
- net GND: vias 0 -> 4
