File: Schematic-PCB/Power-20240325/Power-20240325.kicad_pcb (KiCad board)
At the start: 2 copper layers, 151.3 x 110.3 mm, 60 parts, among them J1 Conn_01x02_Pin, J2 Conn_01x05_Pin, J3 Conn_01x02_Pin, J4 Conn_01x03_Pin, J5 Conn_01x02_Pin, J5 Conn_01x03_Pin, SW1 SW_DPST_x2, SW2 Locker-SW, U1 PIC12F683-IMC

Commit message: 電源基板のPCB完成
DRをお願いします
Parts:
- removed +3.3V, +5V: ~, @2024-Power:OKL-T6-W12N-C
- removed the C1 at (57.0, 76.9)
- removed the C2 at (57.0, 82.4)
- removed the C3 at (114.6, 21.5)
- removed the C4 at (57.0, 91.2)
- removed the C5 at (37.5, 121.7)
- removed the C6 at (39.9, 72.3)
- removed C7: 1000uF, Capacitor_THT:CP_Radial_D10.0mm_P5.00mm
- removed C8: 10uF, Capacitor_SMD:C_0603_1608Metric
- removed D1: LED, LED_THT:LED_D3.0mm
- removed the F1 at (52.1, 118.2)
- removed J2: Conn_01x05_Pin, Connector_PinSocket_2.54mm:PinSocket_1x05_P2.54mm_Vertical
- removed J5: Conn_01x03_Pin, Connector_JST:JST_XH_B3B-XH-A_1x03_P2.50mm_Vertical
- removed the KICKER at (70.0, 79.9)
- removed the LINE at (79.1, 105.4)
- removed the MD at (72.3, 94.6)
- removed MES1: Voltmeter_DC, @2024-Power:VoltMeter
- removed N: NMOS, Package_TO_SOT_SMD:SOT-23
- removed P: PMOS, Package_TO_SOT_SMD:TO-252-2
- removed the R1 at (44.3, 134.4)
- removed R10: 100, Resistor_SMD:R_0603_1608Metric
- removed R12: 1K, Resistor_SMD:R_0603_1608Metric
- removed R13: 10, Resistor_SMD:R_0603_1608Metric
- removed R14: 330, Resistor_SMD:R_0603_1608Metric
- removed R15, R8: 1.2K, Resistor_SMD:R_0603_1608Metric
- removed the R2 at (63.6, 116.7)
- removed the R4 at (35.0, 112.5)
- removed the R5 at (37.5, 120.2)
- removed the R6 at (56.0, 79.6)
- removed the R7 at (58.0, 79.6)
- removed R9: 10K, Resistor_SMD:R_0603_1608Metric
- removed SW2: Locker-SW, @2024-Power:RA1113112R
- removed the U1 at (37.5, 119.4)
- removed U3: ~, Package_TO_SOT_SMD:SOT-89-3
- removed the VIN at (62.1, 130.7)
- C4, C5: moved to B.Cu
- moved R2 73.3 mm to (82.8, 126.0), turned to 0 degrees
- moved R3 73.3 mm to (79.2, 124.2)
- moved R1 73.2 mm to (82.8, 124.2), turned to 180 degrees
- moved C2 72.5 mm to (79.2, 126.0)
- moved U1 69.9 mm to (81.0, 126.0)
- moved C1 68.4 mm to (81.0, 127.8), turned to 0 degrees
- moved C3 44.6 mm to (94.8, 127.8), turned to 0 degrees
- moved + 42.4 mm to (100.0, 112.0)
- moved C4 42.4 mm to (131.5, 144.1)
- moved C5 42.4 mm to (68.5, 144.1)
- moved F1 42.4 mm to (120.0, 132.0)
- moved KICKER 42.4 mm to (81.0, 114.0)
- moved MAIN 42.4 mm to (70.1, 116.1)
- moved MD 42.4 mm to (95.0, 111.7)
- moved SW1 42.4 mm to (100.0, 145.5)
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- renumbered J5 to KICKER, J3 to LINE, J4 to MAIN, J1 to VIN
Routing:
- net (no net): track 178.2 -> 0.00 mm, vias 68 -> 0
- net +5V: track 131.0 -> 55.5 mm, vias 2 -> 3
- net +3.3V: track 71.1 -> 19.6 mm, vias 3 -> 1
- net GND: track 77.2 -> 54.3 mm, vias 10 -> 4
- net VIN: track 9.62 -> 1.95 mm, vias 5 -> 2
- net Net-(U2-Trim): track 12.2 -> 6.35 mm, vias 2 -> 1
- net Net-(U1-Trim): track 3.32 -> 6.35 mm
- net Net-(SW1A-A): vias 0 -> 1
- added copper zone on B.Cu, net Net-(SW1A-A)
- removed copper zone on B.Cu, net (none)
- removed copper zone on F.Cu, net (none)
Other:
- board size 151.3 x 110.3 mm -> 82.9 x 53.9 mm
- board text added: "Power #01"

Commit message: 電源基板のPCBを修正しました
Routing:
- net VIN: track 1.95 -> 3.88 mm, vias 2 -> 3
