File: Schematic-PCB/Power-20240325/Power-20240325.kicad_sch (KiCad schematic)
At the start: 23 parts, among them J1 Conn_01x02_Pin, J2 Conn_01x02_Pin, J3 Conn_01x02_Pin, J4 Conn_01x03_Pin, J5 Conn_01x02_Pin, SW1 SW_DPST_x2

Commit message: MDの回路図/PCBを更新
Parts:
- J5: footprint Connector_JST:JST_XH_B2B-XH-A_1x02_P2.50mm_Vertical -> Connector_JST:JST_XH_S2B-XH-A-1_1x02_P2.50mm_Horizontal
Changed lines of the file:
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@@
 			)
 		)
-		(property "Footprint" "Connector_JST:JST_XH_B2B-XH-A_1x02_P2.50mm_Vertical"
+		(property "Footprint" "Connector_JST:JST_XH_S2B-XH-A-1_1x02_P2.50mm_Horizontal"
 			(at 171.45 113.03 0)
 			(effects

Commit message: ラインセンサ基板のPCBを更新
ちょっと停滞中... ヘルプ求む、
Other:
- moved on the sheet: C1, C2, C3, C4, C5, C6, F1, J1, J2, J3, J4, J5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

Commit message: 電源基板にドリブラーへの電源供給コネクタを追加
Parts:
- added J6: Conn_01x02_Pin, Connector_JST:JST_XH_S2B-XH-A-1_1x02_P2.50mm_Horizontal, symbol Connector:Conn_01x02_Pin
Connections:
- net GND: now also J6.2 (Pin_2)
- net VIN: now also J6.1 (Pin_1)
Other:
- note added: "Dribbler"
Changed lines of the file:
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@@
 	(wire
 		(pts
+			(xy 97.79 168.91) (xy 105.41 168.91)
+		)
+		(stroke
+			(width 0)
+			(type default)
+		)
+	)
+	(wire
+		(pts
 			(xy 31.75 44.45) (xy 31.75 46.99)
 		)
@@
 	(wire
 		(pts
+			(xy 97.79 171.45) (xy 105.41 171.45)
+		)
+		(stroke
+			(width 0)
+			(type default)
+		)
+	)
+	(wire
+		(pts
 			(xy 53.34 71.12) (xy 55.88 71.12)
 		)
@@
 	(wire
 		(pts
+			(xy 105.41 171.45) (xy 105.41 173.99)
+		)
+		(stroke
+			(width 0)
+			(type default)
+		)
+	)
+	(wire
+		(pts
 			(xy 104.14 91.44) (xy 120.65 91.44)
 		)
@@
 	(wire
 		(pts
+			(xy 105.41 166.37) (xy 105.41 168.91)
+		)
+		(stroke
+			(width 0)
+			(type default)
+		)
+	)
+	(wire
+		(pts
 			(xy 76.2 78.74) (xy 76.2 91.44)
 		)
@@
 		)
 	)
+	(text "Dribbler"
+		(exclude_from_sim no)
+		(at 89.662 172.466 0)
+		(effects
+			(font
+				(size 2.54 2.54)
+			)
+			(justify right)
+		)
+	)
 	(text "Line"
 		(exclude_from_sim no)
@@
 	(global_label "VIN"
 		(shape input)
+		(at 105.41 166.37 90)
+		(fields_autoplaced yes)
+		(effects
+			(font
+				(size 1.27 1.27)
+			)
+			(justify left)
+		)
+		(property "Intersheetrefs" "${INTERSHEET_REFS}"
+			(at 105.41 160.0537 90)
+			(effects
+				(font
+					(size 1.27 1.27)
+				)
+				(justify left)
+				(hide yes)
+			)
+		)
+	)
+	(global_label "VIN"
+		(shape input)
 		(at 114.3 30.48 90)
 		(fields_autoplaced yes)
@@
 	(symbol
 		(lib_id "Connector:Conn_01x02_Pin")
+		(at 92.71 168.91 0)
+		(unit 1)
+		(exclude_from_sim no)
+		(in_bom yes)
+		(on_board yes)
+		(dnp no)
+		(fields_autoplaced yes)
+		(property "Reference" "J6"
+			(at 93.345 163.83 0)
+			(effects
+				(font
+					(size 1.27 1.27)
+				)
+			)
+		)
+		(property "Value" "Conn_01x02_Pin"
+			(at 93.345 166.37 0)
+			(effects
+				(font
+					(size 1.27 1.27)
+				)
+			)
+		)
+		(property "Footprint" "Connector_JST:JST_XH_S2B-XH-A-1_1x02_P2.50mm_Horizontal"
+			(at 92.71 168.91 0)
+			(effects
+				(font
+					(size 1.27 1.27)
+				)
+				(hide yes)
+			)
+		)
+		(property "Datasheet" "~"
+			(at 92.71 168.91 0)
+			(effects
+				(font
+					(size 1.27 1.27)
+				)
+				(hide yes)
+			)
+		)
+		(property "Description" "Generic connector, single row, 01x02, script generated"
+			(at 92.71 168.91 0)
+			(effects
+				(font
+					(size 1.27 1.27)
+				)
+				(hide yes)
+			)
+		)
+		(pin "2"
+		)
+		(pin "1"
+		)
+		(instances
+			(project "Power-20240325"
+				(path "/650be7cc-f935-443e-9e0c-9dc933fdca0b"
+					(reference "J6")
+					(unit 1)
+				)
+			)
+		)
+	)
+	(symbol
+		(lib_id "Connector:Conn_01x02_Pin")
 		(at 46.99 119.38 0)
 		(unit 1)
@@
 					(unit 1)
 				)
+			)
+		)
+	)
+	(symbol
+		(lib_id "power:GND")
+		(at 105.41 173.99 0)
+		(unit 1)
+		(exclude_from_sim no)
+		(in_bom yes)
+		(on_board yes)
+		(dnp no)
+		(fields_autoplaced yes)
+		(property "Reference" "#PWR015"
+			(at 105.41 180.34 0)
+			(effects
+				(font
+					(size 1.27 1.27)
+				)
+				(hide yes)
+			)
+		)
+		(property "Value" "GND"
+			(at 105.41 179.07 0)
+			(effects
+				(font
+					(size 1.27 1.27)
+				)
+			)
+		)
+		(property "Footprint" ""
+			(at 105.41 173.99 0)
+			(effects
+				(font
+					(size 1.27 1.27)
+				)
+				(hide yes)
+			)
+		)
+		(property "Datasheet" ""
+			(at 105.41 173.99 0)
+			(effects
+				(font
+					(size 1.27 1.27)
+				)
+				(hide yes)
+			)
+		)
+		(property "Description" "Power symbol creates a global label with name \"GND\" , ground"
+			(at 105.41 173.99 0)
+			(effects
+				(font
+					(size 1.27 1.27)
+				)
+				(hide yes)
+			)
+		)
+		(pin "1"
+		)
+		(instances
+			(project "Power-20240325"
+				(path "/650be7cc-f935-443e-9e0c-9dc933fdca0b"
+					(reference "#PWR015")
+					(unit 1)
+				)

Commit message: update: 電源基板のラインセンサ向け供給コネクタをVHコネクタからXHコネクタに変更した
Parts:
- F1: footprint @2024-Power:Fuse -> @2024TOINIOT2-Power:Fuse
- J1: footprint @2024-Power:VIN -> @2024TOINIOT2-Power:VIN
- J2: footprint @2024-Power:XT30PW-M -> @2024TOINIOT2-Power:XT30PW-M
- J3: footprint Connector_JST:JST_VH_S2P-VH_1x02_P3.96mm_Horizontal -> Connector_JST:JST_XH_B2B-XH-A_1x02_P2.50mm_Vertical
- MES1: footprint @2024-Power:VoltMeter -> @2024TOINIOT2-Power:VoltMeter
- SW1: footprint @2024-Power:RA1113112R -> @2024TOINIOT2-Power:RA1113112R
- U1, U2: footprint @2024-Power:OKL-T6-W12N-C -> @2024TOINIOT2-Power:OKL-T6-W12N-C
Changed lines of the file:
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@@
 			)
 		)
-		(property "Footprint" "@2024-Power:Fuse"
+		(property "Footprint" "@2024TOINIOT2-Power:Fuse"
 			(at 38.1 43.688 90)
 			(effects
@@
 			)
 		)
-		(property "Footprint" "@2024-Power:VIN"
+		(property "Footprint" "@2024TOINIOT2-Power:VIN"
 			(at 24.13 41.91 0)
 			(effects
@@
 			)
 		)
-		(property "Footprint" "@2024-Power:VoltMeter"
+		(property "Footprint" "@2024TOINIOT2-Power:VoltMeter"
 			(at 114.3 35.56 90)
 			(effects
@@
 			)
 		)
-		(property "Footprint" "@2024-Power:OKL-T6-W12N-C"
+		(property "Footprint" "@2024TOINIOT2-Power:OKL-T6-W12N-C"
 			(at 41.91 66.04 0)
 			(effects
@@
 			)
 		)
-		(property "Footprint" "@2024-Power:XT30PW-M"
+		(property "Footprint" "@2024TOINIOT2-Power:XT30PW-M"
 			(at 46.99 119.38 0)
 			(effects
@@
 			)
 		)
-		(property "Footprint" "Connector_JST:JST_VH_S2P-VH_1x02_P3.96mm_Horizontal"
+		(property "Footprint" "Connector_JST:JST_XH_B2B-XH-A_1x02_P2.50mm_Vertical"
 			(at 46.99 140.97 0)
 			(effects
@@
 			)
 		)
-		(property "Footprint" "@2024-Power:RA1113112R"
+		(property "Footprint" "@2024TOINIOT2-Power:RA1113112R"
 			(at 52.07 41.91 0)
 			(effects
@@
 			)
 		)
-		(property "Footprint" "@2024-Power:OKL-T6-W12N-C"
+		(property "Footprint" "@2024TOINIOT2-Power:OKL-T6-W12N-C"
 			(at 92.71 66.04 0)
 			(effects
