File: Schematic-PCB/FPC-MD-Main-20240719/FPC-MD-Main-20240719.kicad_pcb (KiCad board)
At the start: 2 copper layers, 100 x 16 mm, 2 parts, among them J1 Conn_01x15_Pin, J2 Conn_01x15_Pin

Commit message: 色々追加
Routing:
- net Net-(J1-Pin_15): track 0.00 -> 96.0 mm
- net Net-(J1-Pin_14): track 0.00 -> 96.0 mm
- net Net-(J1-Pin_13): track 0.00 -> 96.0 mm
- added copper zone on B.Cu, net (none)
Other:
- outline, holes or cut-outs redrawn
- board text added: "FPC | MD-Main"
