File: Schematic-PCB/FPC-MD-Main-20240719/FPC-MD-Main-20240719.kicad_sch (KiCad schematic)
At the start: 2 parts, among them J1 Conn_01x15_Pin, J2 Conn_01x15_Pin

Commit message: update: FPCケーブル（旧）を裏表導通するように変更した
Parts:
- J1, J2: footprint @2024TOINIOT2-FPC-FFC:FPC-FFC -> @2024TOINIOT2-FPC-FCC:FPC-FFC
Changed lines of the file:
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@@
 			)
 		)
-		(property "Footprint" "@2024TOINIOT2-FPC-FFC:FPC-FFC"
+		(property "Footprint" "@2024TOINIOT2-FPC-FCC:FPC-FFC"
 			(at 85.09 66.04 0)
 			(effects
@@
 		)
 		(instances
-			(project ""
+			(project "FPC-MD-Main-20240719"
 				(path "/d35d1607-b1d6-4b70-8ad5-7c159f549b16"
 					(reference "J1")
@@
 			)
 		)
-		(property "Footprint" "@2024TOINIOT2-FPC-FFC:FPC-FFC"
+		(property "Footprint" "@2024TOINIOT2-FPC-FCC:FPC-FFC"
 			(at 105.41 66.04 0)
 			(effects
