File: Schematic-PCB/Line-002-20241023/Line-002-20241023.kicad_sch (KiCad schematic)
At the start: 208 parts

Commit message: update: ラインセンサ基板ver.002を更新した
回路図をちょっと進めた ∧ PCBをやり始めた
Parts:
- added BZ1: Buzzer, @2024TOINIOT2-Line:PKM13EPYH4000-A0, symbol Device:Buzzer
- added C1, C2, C3: 22pF, symbol Device:C_Small
- added D53: LED01, LED_SMD:LED_0603_1608Metric, symbol Device:LED_Small_Filled
- added D54: LED02, LED_SMD:LED_0603_1608Metric, symbol Device:LED_Small_Filled
- added D55: LED03, LED_SMD:LED_0603_1608Metric, symbol Device:LED_Small_Filled
- added J1: ICSP, symbol Connector_Generic:Conn_02x03_Odd_Even
- added R105: 10K, Resistor_SMD:R_0603_1608Metric, symbol Device:R_Small
- added R106, R107, R108: 330, Resistor_SMD:R_0603_1608Metric, symbol Device:R_Small
- added R109: 1M, symbol Device:R_Small
- added SW1: RESET, symbol Switch:SW_SPST
- added U53: ATmega2560-16A, Package_QFP:TQFP-100_14x14mm_P0.5mm, symbol MCU_Microchip_ATmega:ATmega2560-16A
- added Y1: 16MHz, symbol Device:Crystal_Small
- D1, D10, D11, D12, D13, D14, D15, D16, D17, D18, D19, D2, D20, D21, D22, D23, D24, D25, D26, D27, D28, D29, D3, D30, D31, D32, D33, D34, D35, D36, D37, D38, D39, D4, D40, D41, D42, D43, D44, D45, D46, D47, D48, D49, D5, D50, D51, D52, D6, D7, D8, D9: footprint (none) -> @2024TOINIOT2-Line:LED-3mm
- R1, R10, R100, R101, R102, R103, R104, R11, R12, R13, R14, R15, R16, R17, R18, R19, R2, R20, R21, R22, R23, R24, R25, R26, R27, R28, R29, R3, R30, R31, R32, R33, R34, R35, R36, R37, R38, R39, R4, R40, R41, R42, R43, R44, R45, R46, R47, R48, R49, R5, R50, R51, R52, R53, R54, R55, R56, R57, R58, R59, R6, R60, R61, R62, R63, R64, R65, R66, R67, R68, R69, R7, R70, R71, R72, R73, R74, R75, R76, R77, R78, R79, R8, R80, R81, R82, R83, R84, R85, R86, R87, R88, R89, R9, R90, R91, R92, R93, R94, R95, R96, R97, R98, R99: footprint (none) -> Resistor_SMD:R_0603_1608Metric
Connections:
- net +5V: now also J1.2 (Pin_2), R105.1, U53.10 (VCC), U53.100 (AVCC), U53.31 (VCC), U53.61 (VCC), U53.80 (VCC)
- net GND: now also BZ1.2 (-), C1.2, C2.2, C3.2, D53.1 (K), D54.1 (K), D55.1 (K), J1.6 (Pin_6), SW1.2 (B), U53.11 (GND), U53.32 (GND), U53.62 (GND), U53.81 (GND), U53.99 (GND)
- new net: D53.2 (A), R106.2
- new net: D54.2 (A), R107.2
- new net: D55.2 (A), R108.2
- new net Buzzer: BZ1.1 (+), U53.23 (PB4)
- new net LED01: R106.1, U53.26 (PB7)
- new net LED02: R107.1, U53.25 (PB6)
- new net LED03: R108.1, U53.24 (PB5)
- new net MISO: J1.1 (Pin_1), U53.22 (PB3)
- new net MOSI: J1.4 (Pin_4), U53.21 (PB2)
- new net RESET: C1.1, J1.5 (Pin_5), R105.2, SW1.1 (A), U53.30 (~{RESET})
- new net RX0: U53.2 (PE0)
- new net SCK: J1.3 (Pin_3), U53.20 (PB1)
- new net SS: U53.19 (PB0)
- new net TX0: U53.3 (PE1)
- new net XTAL1: C2.1, R109.1, U53.34 (XTAL1), Y1.1
- new net XTAL2: C3.1, R109.2, U53.33 (XTAL2), Y1.2
- no-connect marks 0 -> 15

Commit message: update: ラインセンサ ver.002 の回路図を進めた
コンパレータを追加
ピンアサインはちょっと悩み中だけどほぼいい感じだと思う...たぶん。
Parts:
- removed R29, R30, R31, R32, R33, R34, R35, R36, R37, R38, R39, R40, R41, R42, R43, R44, R45, R46, R47, R48, R49, R50, R51, R52: Line-PDWN, Resistor_SMD:R_0603_1608Metric, symbol Device:R_Small
- removed U45, U46, U47, U48, U49, U50, U51, U52: ~, @2024TOINIOT2-Line:NJL7502L, symbol @2024-Line:NJL7502L
- added C1, C4, C6, C8: 100nF, symbol Device:C_Small
- added C7: 10uF, symbol Device:C_Small
- added Comp1, Comp2, Comp3, Comp4, Comp5, Comp6, Comp7: ~, symbol @2024-Line:LM339
- added JP1: 160Hz, symbol Jumper:Jumper_2_Small_Open
- added JP2: 16Hz, symbol Jumper:Jumper_2_Small_Open
- added JP3: 1.6Hz, symbol Jumper:Jumper_2_Small_Open
- added R103, R106, R98: 10K, symbol Device:R_Small
- added R104: 100, symbol Device:R_Small
- added R105: 1K, symbol Device:R_Small
- R25, R26, R27, R28: footprint Resistor_SMD:R_0603_1608Metric -> (none)
- renumbered C1 to C3, C3 to C5, R107 to R100, R108 to R101, R109 to R102, R53 to R45, R54 to R46, R55 to R47, R56 to R48, R57 to R49, R58 to R50, R59 to R51, R60 to R52, R61 to R53, R62 to R54, R63 to R55, R64 to R56, R65 to R57, R66 to R58, R67 to R59, R68 to R60, R69 to R61, R70 to R62, R71 to R63, R72 to R64, R73 to R65, R74 to R66, R75 to R67, R76 to R68, R77 to R69, R78 to R70, R79 to R71, R80 to R72, R81 to R73, R82 to R74, R83 to R75, R84 to R76, R85 to R77, R86 to R78, R87 to R79, R88 to R80, R89 to R81, R90 to R82, R91 to R83, R92 to R84, R93 to R85, R94 to R86, R95 to R87, R96 to R88, R97 to R89, R98 to R90, R99 to R91, R100 to R92, R101 to R93, R102 to R94, R103 to R95, R104 to R96, R105 to R97, R106 to R99, U53 to U45
Connections:
- net Line-B-03 is gone; now on net Line-R: U41.1 (Emitter)
- net Line-B-04 is gone; now on net Line-R: U42.1 (Emitter)
- net Line-B-05 is gone; now on net Line-R: U43.1 (Emitter)
- net Line-B-06 is gone; now on net Line-R: U44.1 (Emitter)
- net Line-F-01 is gone; now on net Line-F: R25.1, U25.1 (Emitter)
- net Line-F-05 is gone; now on net Line-F: U29.1 (Emitter)
- net Line-F-06 is gone; now on net Line-L: U30.1 (Emitter)
- net Line-F-07 is gone; now on net Line-L: U31.1 (Emitter)
- net Line-L-01 is gone; now on net Line-L: U32.1 (Emitter)
- net Line-L-02 is gone; now on net Line-L: U33.1 (Emitter)
- net Line-L-03 is gone; now on net Line-L: U34.1 (Emitter)
- net Line-L-04 is gone; now on net Line-B: U35.1 (Emitter)
- net Line-L-05 is gone; now on net Line-B: U36.1 (Emitter)
- net Line-L-06 is gone; now on net Line-B: U37.1 (Emitter)
- net Line-L-07 is gone; now on net Line-B: U38.1 (Emitter)
- net +5V: now also C1.1, C4.1, C6.1, Comp1.3 (VCC), Comp2.3 (VCC), Comp3.3 (VCC), Comp4.3 (VCC), Comp5.3 (VCC), Comp6.3 (VCC), Comp7.3 (VCC), R103.1, R98.1
- net GND: now also C1.2, C4.2, C6.2, C7.2, C8.1, Comp1.12 (GND), Comp2.12 (GND), Comp3.12 (GND), Comp4.12 (GND), Comp5.12 (GND), Comp6.12 (GND), Comp7.12 (GND)
- net Line01: now also U45.5 (PE3), Comp1.5 (2IN+)
- net Line02: now also U45.6 (PE4), Comp1.9 (3IN+)
- net Line03: now also U45.7 (PE5), Comp1.11 (4IN+)
- net Line12: now also U45.50 (PD7)
- net PWM: now reaches U45.1 (PG5)
- net PWM: now also JP1.1 (A), JP2.1 (A), JP3.1 (A)
- net RX2: now reaches U45.12 (PH0)
- net TX2: now reaches U45.13 (PH1)
- net 04: now reaches U45.15 (PH3)
- net 05: now reaches U45.16 (PH4)
- net 06: now reaches U45.17 (PH5)
- net 07: now reaches U45.18 (PH6)
- net 08: now reaches U45.27 (PH7)
- net L-01: now reaches U45.35 (PL0)
- net L-02: now reaches U45.36 (PL1)
- net L-03: now reaches U45.37 (PL2)
- net L-04: now reaches U45.38 (PL3)
- net L-05: now reaches U45.39 (PL4)
- net 09: now reaches U45.40 (PL5)
- net 10: now reaches U45.41 (PL6)
- net 11: now reaches U45.42 (PL7)
- net SCL: now reaches U45.43 (PD0)
- net SCL: now also R103.2
- net SDA: now reaches U45.44 (PD1)
- net SDA: now also R98.2
- net RX1: now reaches U45.45 (PD2)
- net TX1: now reaches U45.46 (PD3)
- net 13: now reaches U45.51 (PG0)
- net 14: now reaches U45.52 (PG1)
- net B-01: now reaches U45.53 (PC0)
- net B-02: now reaches U45.54 (PC1)
- net B-03: now reaches U45.55 (PC2)
- net B-04: now reaches U45.56 (PC3)
- net B-05: now reaches U45.57 (PC4)
- net 15: now reaches U45.58 (PC5)
- net 16: now reaches U45.59 (PC6)
- net 17: now reaches U45.60 (PC7)
- net RX3: now reaches U45.63 (PJ0)
- net TX3: now reaches U45.64 (PJ1)
- net 18: now reaches U45.70 (PG2)
- net 19: now reaches U45.71 (PA7)
- net 20: now reaches U45.72 (PA6)
- net 21: now reaches U45.73 (PA5)
- net R-01: now reaches U45.74 (PA4)
- net R-02: now reaches U45.75 (PA3)
- net R-03: now reaches U45.76 (PA2)
- net R-04: now reaches U45.77 (PA1)
- net R-05: now reaches U45.78 (PA0)
- net 22: now reaches U45.82 (PK7)
- net 23: now reaches U45.83 (PK6)
- net 24: now reaches U45.84 (PK5)
- net Line-F: now reaches U45.94 (PF3)
- net Line-F: now also U26.1 (Emitter), U27.1 (Emitter), U28.1 (Emitter), Comp1.7 (1IN+)
- net 01: now reaches U45.95 (PF2)
- net 01: now also Comp1.2 (2OUT)
- net 02: now reaches U45.96 (PF1)
- net 02: now also Comp1.14 (3OUT)
- net 03: now reaches U45.97 (PF0)
- net 03: now also Comp1.13 (4OUT)
- net at U45.98 (AREF): now also C8.2
- net Line-B-01 renamed Line-B
- net Line-B: now also R27.1
- net Line-B-02 renamed Line-R
- net Line-R: now also R28.1
- net Line-F-02 renamed Line-L
- net Line-L: no longer U26.1 (Emitter)
- removed net Line-F-03: R27.1, U27.1 (Emitter)
- removed net Line-F-04: R28.1, U28.1 (Emitter)
- new net: JP1.2 (B), R104.1
- new net: JP3.2 (B), R106.1
- new net: JP2.2 (B), R105.1
- new net F: Comp1.1 (1OUT)
- new net Threshold: C7.1, Comp1.10 (4IN-), Comp1.4 (2IN-), Comp1.6 (1IN-), Comp1.8 (3IN-), Comp2.10 (4IN-), Comp2.4 (2IN-), Comp2.6 (1IN-), Comp2.8 (3IN-), Comp3.10 (4IN-), Comp3.4 (2IN-), Comp3.6 (1IN-), Comp3.8 (3IN-), Comp4.10 (4IN-), Comp4.4 (2IN-), Comp4.6 (1IN-), Comp4.8 (3IN-), Comp5.10 (4IN-), Comp5.4 (2IN-), Comp5.6 (1IN-), Comp5.8 (3IN-), Comp6.10 (4IN-), Comp6.4 (2IN-), Comp6.6 (1IN-), Comp6.8 (3IN-), Comp7.10 (4IN-), Comp7.4 (2IN-), Comp7.6 (1IN-), Comp7.8 (3IN-), R104.2, R105.2, R106.2
Other:
- moved on the sheet: BZ1, C2, C3, C5, D1, D10, D11, D12, D13, D14, D15, D16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
