File: Schematic-PCB/参考・練習用フォルダ/(練習用) ATmega2560/2023ver/MainBoard_ATMega2560Pro_20230629.kicad_sch (KiCad schematic)
At the start: 39 parts, among them J1 Conn_01x10_Pin, J2 Conn_01x08_Male, J3 Conn_01x04_Female, J4 Conn_01x08_Male, J5 Conn_01x02_Male, J6 Conn_01x20_Male, J7 Conn_01x26_Male, J8 Conn_01x03_Pin, SW1 SW_DPST_x2, SW2 SW_DPST_x2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

Commit message: update: いろいろなKiCadファイルを開いた
Parts:
- removed JP3: Jumper_2_Open, Jumper:SolderJumper-2_P1.3mm_Open_Pad1.0x1.5mm, symbol Jumper:Jumper_2_Open
- added JP3: Jumper_2_Bridged, Jumper:SolderJumper-2_P1.3mm_Bridged_Pad1.0x1.5mm, symbol Jumper:Jumper_2_Bridged
Connections:
- net SS: now also JP3.2 (B)
- net Sig23_BALL-Kicker: now also U1.D48; no longer U1.D49
- net Sig_NeoPixel: now also U1.D49; no longer U1.D11
- net at J1.7 (Pin_7): now also JP3.1 (A)
Other:
- moved on the sheet: U2
