File: Schematic-PCB/Main-002-20241217/Main-20241217.kicad_sch (KiCad schematic)
At the start: 90 parts, among them J1 Conn_PWR, J10 Conn_NeoPixel, J11 Conn_Kicker, J12 Conn_LineUART, J2 CamS3-6, J3 CamS3-4, J4 Pixy 2.1, J5 Conn_MD, J6 Conn_Dribbler, J7 Conn_UI, J8 Conn_NeoPixel, J9 Conn_NeoPixel, SW1 SW_DPDT_x2, SW2 Main_RST, SW3 Cam_RST, SW4 Cam_RST, U1 DEV-16771, U10 TSSP4038, U11 TSSP4038, U12 TSSP4038, U13 TSSP4038, U14 TSSP4038, U15 TSSP4038, U16 TSSP4038, U17 TSSP4038, U18 TSSP4038, U3 TSSP4038, U4 TSSP4038, U5 TSSP4038, U6 TSSP4038, U7 TSSP4038, U8 TSSP4038, U9 TSSP4038

Commit message: update: メインとMDの基板を編集
Parts:
- added Q1, Q2: BSS138, Package_TO_SOT_SMD:SOT-23, symbol Transistor_FET:BSS138
- added R1, R2, R26, R27: 10k, Resistor_SMD:R_0603_1608Metric, symbol Device:R
Connections:
- net +3.3V: now also Q1.1 (G), Q2.1 (G), R1.2, R2.2
- net +5V: now also R26.1, R27.1
- net EN-1: now also J5.8 (Pin_8), U1.7 (RX2); no longer J5.3 (Pin_3), U1.2 (OUT2)
- net EN-2: now also J5.10 (Pin_10), U1.9 (OUT1C); no longer J5.5 (Pin_5), U1.4 (BCLK2)
- net EN-3: now also J5.4 (Pin_4), U1.3 (LRCLK2); no longer J5.7 (Pin_7), U1.6 (OUT1D)
- net EN-4: now also J5.6 (Pin_6), U1.5 (IN2); no longer J5.9 (Pin_9), U1.8 (TX2)
- net PH-1: now also J5.7 (Pin_7), U1.6 (OUT1D); no longer J5.4 (Pin_4), U1.3 (LRCLK2)
- net PH-2: now also J5.9 (Pin_9), U1.8 (TX2); no longer J5.6 (Pin_6), U1.5 (IN2)
- net PH-3: now also J5.3 (Pin_3), U1.2 (OUT2); no longer J5.8 (Pin_8), U1.7 (RX2)
- net PH-4: now also J5.5 (Pin_5), U1.4 (BCLK2); no longer J5.10 (Pin_10), U1.9 (OUT1C)
- new net Line-Main=RX_3.3V: Q1.2 (S), R1.1
- new net Line-Main=RX_5V: Q1.3 (D), R26.2
- new net Line-Main=TX_3.3V: Q2.2 (S), R2.1
- new net Line-Main=TX_5V: Q2.3 (D), R27.2
Other:
- note added: "HIGH"
- note added: "LEVEL CONVERT"
- note added: "LOW"
