File: Schematic-PCB/Line-003-20241222/Line-003-20241222.kicad_pcb (KiCad board)
At the start: 4 copper layers, 196 x 194.2 mm, 220 parts, among them J1 ICSP, J2 VIN, U45 ATmega2560-16A, U62 ATmega2560 Pro Board, Y1 16MHz

Commit message: update: ラインセンサ基板 ver.003 を更新した
回路図のDRをした
いろいろ問題点ありそうだから、明日もう一回DRし直してからPCBいこか
出来れば明日、無理なら明後日ぐらいまでに必ず完成させよう！！
Parts:
- removed BZ1: Buzzer, @2024TOINIOT2-Line:PKM13EPYH4000-A0
- removed D49, D50, D51, D52: Wh/Rd, @2024TOINIOT2-Line:LED-3mm
- removed D53: LED01, LED_SMD:LED_0603_1608Metric
- removed D54: LED02, LED_SMD:LED_0603_1608Metric
- removed D55: LED03, LED_SMD:LED_0603_1608Metric
- removed D56: PWR, LED_SMD:LED_0603_1608Metric
- removed J2: VIN, Connector_JST:JST_VH_B2P-VH-B_1x02_P3.96mm_Vertical
- removed R89: 1K, Resistor_SMD:R_0603_1608Metric
- removed R90: 10K, Resistor_SMD:R_0603_1608Metric
- removed R91: 330, Resistor_SMD:R_0603_1608Metric
- removed REF** (x11): MountingHole_3.2mm_M3, MountingHole:MountingHole_3.2mm_M3
- removed U62: ATmega2560 Pro Board, @2024TOINIOT2-Line:ATmega2560Pro Board
- removed Y1: 16MHz, @2024TOINIOT2-Line:AL4BT
- added C10: 100nF, Capacitor_SMD:C_0603_1608Metric, F.Cu at (170.1, 62.6)
- added C11: 100nF, Capacitor_SMD:C_0603_1608Metric, F.Cu at (170.1, 65.1)
- added C12: 100nF, Capacitor_SMD:C_0603_1608Metric, F.Cu at (170.1, 67.6)
- added C13: 100nF, Capacitor_SMD:C_0603_1608Metric, F.Cu at (174.1, 40.0)
- added C17: 100nF, Capacitor_SMD:C_0603_1608Metric, F.Cu at (174.1, 42.5)
- added C18: 100nF, Capacitor_SMD:C_0603_1608Metric, F.Cu at (174.1, 45.0)
- added C19: 100nF, Capacitor_SMD:C_0603_1608Metric, F.Cu at (174.1, 47.5)
- added C20: 100nF, Capacitor_SMD:C_0603_1608Metric, F.Cu at (174.1, 50.0)
- added C21: 100nF, Capacitor_SMD:C_0603_1608Metric, F.Cu at (174.1, 52.5)
- added C22: 100nF, Capacitor_SMD:C_0603_1608Metric, F.Cu at (174.1, 55.1)
- added C24: 10uF, Capacitor_SMD:C_0805_2012Metric, F.Cu at (188.2, 129.3)
- added C25: 10uF, Capacitor_SMD:C_0805_2012Metric, F.Cu at (188.2, 132.3)
- added JP10: Jumper_2_Small_Open, Jumper:SolderJumper-2_P1.3mm_Open_Pad1.0x1.5mm, F.Cu at (183.8, 133.2)
- added JP4: 160Hz, Jumper:SolderJumper-2_P1.3mm_Open_Pad1.0x1.5mm, F.Cu at (179.4, 129.7)
- added JP5: 16Hz, Jumper:SolderJumper-2_P1.3mm_Open_Pad1.0x1.5mm, F.Cu at (179.4, 133.2)
- added JP6: 1.6Hz, Jumper:SolderJumper-2_P1.3mm_Open_Pad1.0x1.5mm, F.Cu at (183.8, 119.0)
- added JP7: Jumper_2_Small_Open, Jumper:SolderJumper-2_P1.3mm_Open_Pad1.0x1.5mm, F.Cu at (183.8, 122.6)
- added JP8: Jumper_2_Small_Open, Jumper:SolderJumper-2_P1.3mm_Open_Pad1.0x1.5mm, F.Cu at (183.8, 126.2)
- added JP9: Jumper_2_Small_Open, Jumper:SolderJumper-2_P1.3mm_Open_Pad1.0x1.5mm, F.Cu at (183.8, 129.7)
- added U46: ~, @2024TOINIOT2-Line:NJL7502L, F.Cu at (174.6, 106.7)
- added U47: LM393, Package_SO:SOIC-8_3.9x4.9mm_P1.27mm, F.Cu at (181.5, 81.2)
- added U48: LM393, Package_SO:SOIC-8_3.9x4.9mm_P1.27mm, F.Cu at (181.5, 87.7)
- added U49: LM393, Package_SO:SOIC-8_3.9x4.9mm_P1.27mm, F.Cu at (181.5, 94.3)
- added U50: LM393, Package_SO:SOIC-8_3.9x4.9mm_P1.27mm, F.Cu at (181.5, 100.9)
- added U51: LM393, Package_SO:SOIC-8_3.9x4.9mm_P1.27mm, F.Cu at (181.5, 107.5)
- added U52: LM393, Package_SO:SOIC-8_3.9x4.9mm_P1.27mm, F.Cu at (181.5, 114.0)
- added U53: LM393, Package_SO:SOIC-8_3.9x4.9mm_P1.27mm, F.Cu at (189.9, 81.2)
- added U54: LM393, Package_SO:SOIC-8_3.9x4.9mm_P1.27mm, F.Cu at (189.9, 87.7)
- added U55: LM393, Package_SO:SOIC-8_3.9x4.9mm_P1.27mm, F.Cu at (189.9, 94.3)
- added U56: LM393, Package_SO:SOIC-8_3.9x4.9mm_P1.27mm, F.Cu at (189.9, 100.9)
- added U57: LM393, Package_SO:SOIC-8_3.9x4.9mm_P1.27mm, F.Cu at (189.9, 107.5)
- added U58: LM393, Package_SO:SOIC-8_3.9x4.9mm_P1.27mm, F.Cu at (189.9, 114.0)
- added U59: LM393, Package_SO:SOIC-8_3.9x4.9mm_P1.27mm, F.Cu at (198.4, 81.2)
- added U63: LM393, Package_SO:SOIC-8_3.9x4.9mm_P1.27mm, F.Cu at (198.4, 87.7)
- added U64: LM393, Package_SO:SOIC-8_3.9x4.9mm_P1.27mm, F.Cu at (198.4, 94.3)
- added U65: ATmega2560 Pro Board, @2024TOINIOT2-Line:ATmega2560Pro Board, F.Cu at (140.6, 58.3)
- C3, C4, C6: value 22pF -> 100nF
- C8: value 1000uF -> 100nF
- C9: value 10uF -> 100nF; footprint Capacitor_SMD:C_0805_2012Metric -> Capacitor_SMD:C_0603_1608Metric
- D1, D10, D11, D12, D13, D14, D15, D16, D17, D18, D19, D2, D20, D21, D22, D23, D24, D25, D26, D27, D28, D29, D3, D4, D5, D6, D7, D8, D9, U1, U10, U11, U12, U13, U14, U15, U16, U17, U18, U19, U2, U20, U21, U22, U23, U24, U25, U26, U27, U28, U29, U3, U4, U5, U6, U7, U8, U9: moved to F.Cu
- D47: value Wh/Rd -> LED01; footprint @2024TOINIOT2-Line:LED-3mm -> LED_SMD:LED_0603_1608Metric
- D48: value Wh/Rd -> PWR; footprint @2024TOINIOT2-Line:LED-3mm -> LED_SMD:LED_0603_1608Metric
- J1: value ICSP -> VIN; footprint Connector_PinHeader_2.54mm:PinHeader_2x03_P2.54mm_Vertical -> Connector_JST:JST_VH_B2P-VH-B_1x02_P3.96mm_Vertical
- R27, R28: value Line-PDWN -> Line-PDWN2
- R29, R30: value 75 -> Line-PDWN2
- R77, R78: value 75 -> 1K
- R79: value 75 -> 330
- R80: value 75 -> 100
- R81: value 10K -> 1K
- R83: value 330 -> 100
- R84: value 330 -> 1K
- R85: value 330 -> 10K
- R86: value 1M -> 100
- R87: value 10K -> 100
- R88: value 100 -> 330
- U45: value ATmega2560-16A -> ~; footprint Package_QFP:TQFP-100_14x14mm_P0.5mm -> @2024TOINIOT2-Line:NJL7502L
- moved U25 250.9 mm to (164.1, 80.4), turned to 0 degrees
- moved U5 247.6 mm to (148.4, 101.4), turned to 0 degrees
- moved U6 247.5 mm to (148.4, 106.7), turned to 0 degrees
- moved U4 243.7 mm to (148.4, 96.2), turned to 0 degrees
- moved U7 243.6 mm to (148.4, 111.9), turned to 0 degrees
- moved U26 242.7 mm to (164.1, 85.7), turned to 0 degrees
- moved U27 236.4 mm to (164.1, 90.9), turned to 0 degrees
- moved U8 236.1 mm to (148.4, 117.2), turned to 0 degrees
- moved U3 236.0 mm to (148.4, 90.9), turned to 0 degrees
- moved U29 236.0 mm to (164.1, 101.4), turned to 0 degrees
- moved U28 233.8 mm to (164.1, 96.2), turned to 0 degrees
- moved U24 231.1 mm to (158.9, 117.2), turned to 0 degrees
- moved D23 230.6 mm to (126.7, 113.2), turned to 0 degrees
- moved D24 229.5 mm to (126.7, 118.7), turned to 0 degrees
- moved D22 229.2 mm to (126.7, 107.8), turned to 0 degrees
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Connections:
- C1 pad 2: Net-(U45-AREF) -> +5V
- C2 pad 1: +5V -> GND
- C2 pad 2: GND -> +5V
- C3 pad 1: XTAL1 -> GND
- C3 pad 2: GND -> +5V
- C4 pad 1: RESET -> GND
- C4 pad 2: GND -> +5V
- C5 pad 1: +5V -> GND
- C5 pad 2: GND -> +5V
- C6 pad 1: XTAL2 -> GND
- C6 pad 2: GND -> +5V
- C7 pad 1: +5V -> GND
- C7 pad 2: GND -> +5V
- C8 pad 1: +5V -> GND
- C8 pad 2: GND -> +5V
- C9 pad 1: Threshold -> GND
- C9 pad 2: GND -> +5V
- J1 pad 1: MISO -> +5V
- J1 pad 2: +5V -> GND
- R25 pad 1: Line-F -> Line25
- R26 pad 1: Line-L -> Line26
- R27 pad 1: Line-B -> Line-F
- R28 pad 1: Line-R -> Line-L
- R29 pad 1: +5V -> Line-B
- R29 pad 2: Net-(D1-A) -> GND
- R30 pad 1: +5V -> Line-R
- R30 pad 2: Net-(D2-A) -> GND
- R31 pad 2: Net-(D3-A) -> Net-(D1-A)
- R32 pad 2: Net-(D4-A) -> Net-(D2-A)
- R33 pad 2: Net-(D5-A) -> Net-(D3-A)
- R34 pad 2: Net-(D6-A) -> Net-(D4-A)
- R35 pad 2: Net-(D7-A) -> Net-(D5-A)
- R36 pad 2: Net-(D8-A) -> Net-(D6-A)
- R37 pad 2: Net-(D9-A) -> Net-(D7-A)
- R38 pad 2: Net-(D10-A) -> Net-(D8-A)
- R39 pad 2: Net-(D11-A) -> Net-(D9-A)
- R40 pad 2: Net-(D12-A) -> Net-(D10-A)
- R41 pad 2: Net-(D13-A) -> Net-(D11-A)
- R42 pad 2: Net-(D14-A) -> Net-(D12-A)
- R43 pad 2: Net-(D15-A) -> Net-(D13-A)
- R44 pad 2: Net-(D16-A) -> Net-(D14-A)
- R45 pad 2: Net-(D17-A) -> Net-(D15-A)
- R46 pad 2: Net-(D18-A) -> Net-(D16-A)
- R47 pad 2: Net-(D19-A) -> Net-(D17-A)
- R48 pad 2: Net-(D20-A) -> Net-(D18-A)
- R49 pad 2: Net-(D21-A) -> Net-(D19-A)
- R50 pad 2: Net-(D22-A) -> Net-(D20-A)
- R51 pad 2: Net-(D23-A) -> Net-(D21-A)
- R52 pad 2: Net-(D24-A) -> Net-(D22-A)
- R53 pad 2: Net-(D25-A) -> Net-(D23-A)
- R54 pad 2: Net-(D26-A) -> Net-(D24-A)
- R55 pad 2: Net-(D27-A) -> Net-(D25-A)
- R56 pad 2: Net-(D28-A) -> Net-(D26-A)
- R57 pad 2: Net-(D29-A) -> Net-(D27-A)
- R58 pad 2: Net-(D30-A) -> Net-(D28-A)
- R59 pad 2: Net-(D31-A) -> Net-(D29-A)
- R60 pad 2: Net-(D32-A) -> Net-(D30-A)
- R61 pad 2: Net-(D33-A) -> Net-(D31-A)
- R62 pad 2: Net-(D34-A) -> Net-(D32-A)
- R63 pad 2: Net-(D35-A) -> Net-(D33-A)
- R64 pad 2: Net-(D36-A) -> Net-(D34-A)
- R65 pad 2: Net-(D37-A) -> Net-(D35-A)
- R66 pad 2: Net-(D38-A) -> Net-(D36-A)
- R67 pad 2: Net-(D39-A) -> Net-(D37-A)
- R68 pad 2: Net-(D40-A) -> Net-(D38-A)
- R69 pad 2: Net-(D41-A) -> Net-(D39-A)
- R70 pad 2: Net-(D42-A) -> Net-(D40-A)
- R71 pad 2: Net-(D43-A) -> Net-(D41-A)
- R72 pad 2: Net-(D44-A) -> Net-(D42-A)
- R73 pad 2: Net-(D45-A) -> Net-(D43-A)
- R74 pad 2: Net-(D46-A) -> Net-(D44-A)
- R75 pad 2: Net-(D47-A) -> Net-(D45-A)
- R76 pad 2: Net-(D48-A) -> Net-(D46-A)
- R77 pad 2: Net-(D49-A) -> SDA
- R78 pad 2: Net-(D50-A) -> SCL
- R79 pad 1: +5V -> LED_BUILTIN
- R79 pad 2: Net-(D51-A) -> Net-(D47-A)
- R80 pad 1: +5V -> Net-(JP1-B)
- R80 pad 2: Net-(D52-A) -> Threshold
- R81 pad 1: +5V -> Net-(JP2-B)
- R81 pad 2: RESET -> Threshold
- R82 pad 1: +5V -> Net-(JP3-B)
- R82 pad 2: SDA -> Threshold
- R83 pad 1: LED01 -> Net-(JP4-B)
- R83 pad 2: Net-(D53-A) -> Threshold2
- R84 pad 1: LED02 -> Net-(JP5-B)
- R84 pad 2: Net-(D54-A) -> Threshold2
- R85 pad 1: LED03 -> Net-(JP6-B)
- R85 pad 2: Net-(D55-A) -> Threshold2
- R86 pad 1: XTAL1 -> Net-(J2-Pin_3)
- R86 pad 2: XTAL2 -> Net-(JP9-A)
- R87 pad 1: +5V -> Net-(J2-Pin_4)
- R87 pad 2: SCL -> Net-(JP10-A)
- R88 pad 1: Net-(JP1-B) -> Net-(D48-A)
- R88 pad 2: Threshold -> +5V
- U25 pad 1: Line-F -> Line25
- U26 pad 1: Line-F -> Line26
- U30 pad 1: Line-L -> Line-F
- U31 pad 1: Line-L -> Line-F
- U35 pad 1: Line-B -> Line-L
- U36 pad 1: Line-B -> Line-L
- U40 pad 1: Line-R -> Line-B
- U41 pad 1: Line-R -> Line-B
- U45 pad 1: PWM -> Line-R
- U45 pad 2: RX0 -> +5V
Routing:
- net Line-F: track 46.8 -> 0.00 mm
- removed copper zone on In1.Cu, net +5V
- removed copper zone on B.Cu, net GND
- removed copper zone on F.Cu, net GND
Other:
- board size 196 x 194.2 mm -> 196 x 193.6 mm

Commit message: add: ラインセンサ基板 ver.003を更新した
あと3Dプリンタ印刷用ファイルも追加した
Parts:
- removed C24, C25: 10uF, Capacitor_SMD:C_0805_2012Metric
- removed U63, U64: LM393, Package_SO:SOIC-8_3.9x4.9mm_P1.27mm
- removed U65: ATmega2560 Pro Board, @2024TOINIOT2-Line:ATmega2560Pro Board
- added C14: 100nF, Capacitor_SMD:C_0603_1608Metric, B.Cu at (2.00, 84.0)
- added C15: 100nF, Capacitor_SMD:C_0603_1608Metric, B.Cu at (85.5, 0.50)
- added C16: 100nF, Capacitor_SMD:C_0603_1608Metric, F.Cu at (181.9, 73.6)
- added J2: Conn_MD, @2024TOINIOT2-Line:Connector-MD, F.Cu at (29.0, -14.0)
- added U60: LM393, Package_SO:SOIC-8_3.9x4.9mm_P1.27mm, B.Cu at (49.0, -43.4)
- added U61: LM393, Package_SO:SOIC-8_3.9x4.9mm_P1.27mm, B.Cu at (23.2, -61.2)
- added U62: ATmega2560 Pro Board, @2024TOINIOT2-Line:ATmega2560Pro Board, F.Cu at (-68.0, 0.00)
- C1, C10, C11, C12, C13, C2, C3, C4, C5, C6, C7, C8, C9, D1, D10, D11, D12, D13, D14, D15, D16, D17, D18, D19, D2, D20, D21, D22, D23, D24, D25, D26, D27, D28, D29, D3, D30, D31, D32, D33, D34, D35, D36, D37, D38, D39, D4, D40, D41, D42, D43, D44, D45, D46, D47, D48, D5, D6, D7, D8, D9, R1, R10, R11, R12, R13, R14, R15, R16, R17, R18, R19, R2, R20, R21, R22, R23, R24, R25, R26, R3, R31, R32, R33, R34, R35, R36, R37, R38, R39, R4, R40, R41, R42, R43, R44, R45, R46, R47, R48, R49, R5, R50, R51, R52, R53, R54, R55, R56, R57, R58, R59, R6, R60, R61, R62, R63, R64, R65, R66, R67, R68, R69, R7, R70, R71, R72, R73, R74, R75, R76, R8, R9, U1, U10, U11, U12, U13, U14, U15, U16, U17, U18, U19, U2, U20, U21, U22, U23, U24, U25, U26, U27, U28, U29, U3, U30, U31, U32, U33, U34, U35, U36, U37, U38, U39, U4, U40, U41, U42, U43, U44, U45, U46, U47, U48, U49, U5, U50, U51, U52, U53, U54, U55, U56, U57, U58, U59, U6, U7, U8, U9: moved to B.Cu
- C20: value 100nF -> 1000uF; footprint Capacitor_SMD:C_0603_1608Metric -> Capacitor_THT:CP_Radial_D10.0mm_P5.00mm
- C21, C22: value 100nF -> 10uF; footprint Capacitor_SMD:C_0603_1608Metric -> Capacitor_SMD:C_0805_2012Metric
- J1: footprint Connector_JST:JST_VH_B2P-VH-B_1x02_P3.96mm_Vertical -> Connector_JST:JST_XH_B2B-XH-A_1x02_P2.50mm_Vertical
- moved R62 293.6 mm to (-88.2, -20.4), turned to -13 degrees
- moved R63 293.0 mm to (-90.1, -8.67), turned to -5.5 degrees
- moved U32 293.0 mm to (-92.2, -24.7), turned to -15 degrees
- moved R64 292.7 mm to (-90.4, -3.16), turned to -2 degrees
- moved R65 290.3 mm to (-90.1, 8.67), turned to 5.5 degrees
- moved R66 287.0 mm to (-88.2, 20.4), turned to 13 degrees
- moved U51 281.5 mm to (-78.7, 0.00), turned to -90 degrees
- moved U33 279.9 mm to (-94.7, -12.5), turned to -7.5 degrees
- moved U34 278.4 mm to (-95.5, -0.00)
- moved U31 276.1 mm to (-24.7, -89.4), turned to -135 degrees
- moved U35 275.5 mm to (-94.7, 12.5), turned to 7.5 degrees
- moved U50 271.4 mm to (-63.6, -15.7), turned to -103.847 degrees
- moved U36 271.2 mm to (-92.2, 24.7), turned to 15 degrees
- moved U49 268.5 mm to (-49.0, -43.4), turned to -131.539 degrees
- moved R61 261.6 mm to (-26.0, -83.8), turned to 49.5 degrees
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Connections:
- C17 pad 1: GND -> +5V
- C17 pad 2: +5V -> GND
- C18 pad 2: +5V -> RESET
- C21 pad 1: GND -> Threshold
- C21 pad 2: RESET -> GND
- C22 pad 1: +5V -> Threshold2
- U47 pad 5: Line02 -> Line-F
- U47 pad 6: Th -> Th2
- U47 pad 7: 02 -> F
- U48 pad 1: 03 -> 02
- U48 pad 3: Line03 -> Line02
- U48 pad 5: Line04 -> Line03
- U48 pad 7: 04 -> 03
- U49 pad 1: 05 -> 04
- U49 pad 3: Line05 -> Line04
- U49 pad 5: Line06 -> Line05
- U49 pad 7: 06 -> 05
- U50 pad 1: 07 -> 06
- U50 pad 3: Line07 -> Line06
- U50 pad 5: Line08 -> Line07
- U50 pad 7: 08 -> 07
- U51 pad 1: 09 -> L
- U51 pad 2: Th -> Th2
- U51 pad 3: Line09 -> Line-L
- U51 pad 5: Line10 -> Line08
- U51 pad 7: 10 -> 08
- U52 pad 1: 11 -> 09
- U52 pad 3: Line11 -> Line09
- U52 pad 5: Line12 -> Line10
- U52 pad 7: 12 -> 10
- U53 pad 1: 13 -> 11
- U53 pad 3: Line13 -> Line11
- U53 pad 5: Line14 -> Line12
- U53 pad 7: 14 -> 12
- U54 pad 1: 15 -> 13
- U54 pad 3: Line15 -> Line13
- U54 pad 5: Line16 -> Line14
- U54 pad 7: 16 -> 14
- U55 pad 1: 17 -> B
- U55 pad 2: Th -> Th2
- U55 pad 3: Line17 -> Line-B
- U55 pad 5: Line18 -> Line15
- U55 pad 7: 18 -> 15
- U56 pad 1: 19 -> 16
- U56 pad 3: Line19 -> Line16
- U56 pad 5: Line20 -> Line17
- U56 pad 7: 20 -> 17
- U57 pad 1: 21 -> 18
- U57 pad 3: Line21 -> Line18
- U57 pad 5: Line22 -> Line19
- U57 pad 7: 22 -> 19
- U58 pad 1: 23 -> R
- U58 pad 2: Th -> Th2
- U58 pad 3: Line23 -> Line-R
- U58 pad 5: Line24 -> Line20
- U58 pad 7: 24 -> 20
- U59 pad 1: 25 -> 21
- U59 pad 3: Line25 -> Line21
- U59 pad 5: Line26 -> Line22
- U59 pad 7: 26 -> 22
Routing:
- net +5V: track 0.00 -> 102.9 mm, vias 0 -> 22
- net Line-F: track 0.00 -> 56.6 mm
- net Line-L: track 0.00 -> 49.3 mm
- net Line-B: track 0.00 -> 49.3 mm
- net Line-R: track 0.00 -> 49.3 mm
- net Line15: track 0.00 -> 21.5 mm
- net Line20: track 0.00 -> 17.1 mm
- net Line26: track 0.00 -> 9.40 mm
- net Line24: track 0.00 -> 9.40 mm
- net Line03: track 0.00 -> 9.40 mm
- net Line22: track 0.00 -> 9.40 mm
- net Line05: track 0.00 -> 9.40 mm
- net Line19: track 0.00 -> 9.40 mm
- net Line07: track 0.00 -> 9.40 mm
- net Line17: track 0.00 -> 9.40 mm
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- added copper zone on In1.Cu, net +5V
- added copper zone on B.Cu, net GND
- added copper zone on F.Cu, net GND
Other:
- outline, holes or cut-outs redrawn

Commit message: update: ラインセンサ基板の回路とPCBを更新した
閾値用PWMの周波数選択用のジャンパの削除
基板外形の更新
など
Parts:
- removed JP1, JP4: 160Hz, Jumper:SolderJumper-2_P1.3mm_Open_Pad1.0x1.5mm
- removed JP2, JP5: 16Hz, Jumper:SolderJumper-2_P1.3mm_Open_Pad1.0x1.5mm
- removed JP3, JP6: 1.6Hz, Jumper:SolderJumper-2_P1.3mm_Open_Pad1.0x1.5mm
- removed R80, R83: 100, Resistor_SMD:R_0603_1608Metric
- removed R82, R85: 10K, Resistor_SMD:R_0603_1608Metric
- added REF**: MountingHole_3.2mm_M3, MountingHole:MountingHole_3.2mm_M3, F.Cu at (-47.7, -25.0)
- added REF**: MountingHole_3.2mm_M3, MountingHole:MountingHole_3.2mm_M3, F.Cu at (31.2, 87.4)
- added REF**: MountingHole_3.2mm_M3, MountingHole:MountingHole_3.2mm_M3, F.Cu at (29.7, -92.1)
- added REF**: MountingHole_3.2mm_M3, MountingHole:MountingHole_3.2mm_M3, F.Cu at (79.4, 25.6)
- added REF**: MountingHole_3.2mm_M3, MountingHole:MountingHole_3.2mm_M3, F.Cu at (-88.0, 31.8)
- added REF**: MountingHole_3.2mm_M3, MountingHole:MountingHole_3.2mm_M3, F.Cu at (-38.3, 37.7)
- added REF**: MountingHole_3.2mm_M3, MountingHole:MountingHole_3.2mm_M3, F.Cu at (-80.6, -25.6)
- added REF**: MountingHole_3.2mm_M3, MountingHole:MountingHole_3.2mm_M3, F.Cu at (-26.2, 80.0)
- added REF**: MountingHole_3.2mm_M3, MountingHole:MountingHole_3.2mm_M3, F.Cu at (-30.9, -92.1)
- added REF**: MountingHole_3.2mm_M3, MountingHole:MountingHole_3.2mm_M3, F.Cu at (37.1, -37.7)
- added REF**: MountingHole_3.2mm_M3, MountingHole:MountingHole_3.2mm_M3, F.Cu at (-32.4, 87.4)
- added REF**: MountingHole_3.2mm_M3, MountingHole:MountingHole_3.2mm_M3, F.Cu at (79.4, -25.6)
- added REF**: MountingHole_3.2mm_M3, MountingHole:MountingHole_3.2mm_M3, F.Cu at (-82.3, -11.4)
- added REF**: MountingHole_3.2mm_M3, MountingHole:MountingHole_3.2mm_M3, F.Cu at (37.1, 37.7)
- added REF**: MountingHole_3.2mm_M3, MountingHole:MountingHole_3.2mm_M3, F.Cu at (-38.3, -37.7)
- added REF**: MountingHole_3.2mm_M3, MountingHole:MountingHole_3.2mm_M3, F.Cu at (46.5, -25.0)
- added REF**: MountingHole_3.2mm_M3, MountingHole:MountingHole_3.2mm_M3, F.Cu at (46.5, 25.0)
- added REF**: MountingHole_3.2mm_M3, MountingHole:MountingHole_3.2mm_M3, F.Cu at (86.8, 31.8)
- added REF**: MountingHole_3.2mm_M3, MountingHole:MountingHole_3.2mm_M3, F.Cu at (86.8, -31.8)
- added REF**: MountingHole_3.2mm_M3, MountingHole:MountingHole_3.2mm_M3, F.Cu at (-47.7, 25.0)
- added REF**: MountingHole_3.2mm_M3, MountingHole:MountingHole_3.2mm_M3, F.Cu at (-80.6, 25.6)
- added REF**: MountingHole_3.2mm_M3, MountingHole:MountingHole_3.2mm_M3, F.Cu at (-88.0, -31.8)
- added REF**: MountingHole_3.2mm_M3, MountingHole:MountingHole_3.2mm_M3, F.Cu at (25.1, 80.0)
- JP10, JP7, JP8, JP9, R86, R87, R88: moved to B.Cu
- moved R86 259.8 mm to (-44.6, -1.00), turned to 180 degrees
- moved JP9 259.3 mm to (-48.1, -1.00), turned to 180 degrees
- moved R87 258.1 mm to (-44.6, 7.00), turned to 180 degrees
- moved JP10 257.5 mm to (-48.1, 7.00), turned to 180 degrees
- moved JP8 252.4 mm to (-44.6, 4.50), turned to 180 degrees
- moved JP7 252.2 mm to (-44.6, 1.50), turned to 180 degrees
- moved C21 240.0 mm to (14.8, 0.31)
- moved C22 240.0 mm to (14.8, 3.32)
- moved R79 209.4 mm to (10.6, 0.06)
- moved R77 207.8 mm to (6.55, 7.59)
- moved R78 207.8 mm to (6.55, 10.1)
- moved R84 204.1 mm to (10.6, 5.08)
- moved R81 202.4 mm to (10.6, 2.57)
- moved R28 195.3 mm to (6.55, 0.06)
- moved R29 195.3 mm to (6.55, 2.57)
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Connections:
- R81 pad 1: Net-(JP2-B) -> PWM
- R84 pad 1: Net-(JP5-B) -> PWM2
Routing:
- net RX: track 0.00 -> 26.6 mm, vias 0 -> 1
- net TX: track 0.00 -> 18.4 mm, vias 0 -> 1
- net Net-(J2-Pin_4): track 0.00 -> 11.6 mm
- net Net-(J2-Pin_3): track 0.00 -> 11.6 mm
- net +5V: track 102.9 -> 105.2 mm, vias 22 -> 23
- net Net-(JP9-A): track 0.00 -> 2.03 mm
- net Net-(JP10-A): track 0.00 -> 2.03 mm
- net Line15: vias 0 -> 1
- net Line11: vias 0 -> 1
- net Line17: vias 0 -> 1
- net Line19: vias 0 -> 1
- net Line13: vias 0 -> 1
- net Line01: vias 0 -> 1
- net SDA: vias 0 -> 1
- net SCL: vias 0 -> 1
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Other:
- outline, holes or cut-outs redrawn
- board text added: "+"
- board text added: "G"
- board text added: "RX"
- board text added: "TX"
