File: Schematic-PCB/FPC-MD-Main-002-20241229/FPC-MD-Main-002-20241229.kicad_pcb (KiCad board)
At the start: 2 copper layers, 0 parts

Commit message: update: FPCケーブルの補強材に関する注釈をつけて発注用ファイルを作成した
次回発注があるならこれを使うかもしれない
ただしケーブル本体の長さに関しては要確認（補強材の長さを考えてないため）
Parts:
- added J1: Conn_01x15_Pin, @2024TOINIOT2-FPC-FCC:FPC-FFC, F.Cu at (98.0, 0.00)
- added J2: Conn_01x15_Pin, @2024TOINIOT2-FPC-FCC:FPC-FFC, F.Cu at (2.00, 0.00)
Routing:
- net Net-(J1-Pin_9): track 0.00 -> 96.0 mm
- net Net-(J1-Pin_8): track 0.00 -> 96.0 mm
- net Net-(J1-Pin_7): track 0.00 -> 96.0 mm
- net Net-(J1-Pin_6): track 0.00 -> 96.0 mm
- net Net-(J1-Pin_5): track 0.00 -> 96.0 mm
- net Net-(J1-Pin_4): track 0.00 -> 96.0 mm
- net Net-(J1-Pin_3): track 0.00 -> 96.0 mm
- net Net-(J1-Pin_2): track 0.00 -> 96.0 mm
- net Net-(J1-Pin_15): track 0.00 -> 96.0 mm
- net Net-(J1-Pin_14): track 0.00 -> 96.0 mm
- net Net-(J1-Pin_13): track 0.00 -> 96.0 mm
- net Net-(J1-Pin_12): track 0.00 -> 96.0 mm
- net Net-(J1-Pin_11): track 0.00 -> 96.0 mm
- net Net-(J1-Pin_10): track 0.00 -> 96.0 mm
- net Net-(J1-Pin_1): track 0.00 -> 96.0 mm
Other:
- board outline added: 100 x 16 mm
- board text added: "FPC | MD-Main | 005"
