File: Schematic-PCB/Main-003-20241229/Main-003-20241229.kicad_sch (KiCad schematic)
At the start: 88 parts, among them J1 Conn_PWR, J10 Conn_UI, J2 Conn_NeoPixel, J3 Conn_NeoPixel, J4 Conn_NeoPixel, J5 CamS3-6, J6 CamS3-4, J7 Pixy 2.1, J8 Conn_MD, J9 Conn_Dribbler, SW1 Main_RST, SW2 Cam_RST, SW3 Cam_RST, SW4 SW_DPDT_x2, U1 TSSP4038, U10 TSSP4038, U11 TSSP4038, U12 TSSP4038, U13 TSSP4038, U14 TSSP4038, U15 TSSP4038, U16 TSSP4038, U17 DEV-16771, U2 TSSP4038, U3 TSSP4038, U4 TSSP4038, U5 TSSP4038, U6 TSSP4038, U7 TSSP4038, U8 TSSP4038, U9 TSSP4038

Commit message: update: メイン基板のPCBを更新した
Parts:
- added JP1, JP2: Jumper_2_Small_Open, Jumper:SolderJumper-2_P1.3mm_Open_Pad1.0x1.5mm, symbol Jumper:Jumper_2_Small_Open
Connections:
- net +3.3V: now also JP2.2 (B); no longer R20.1
- net +5V: now also JP1.2 (B); no longer R19.1
- net EN-1: now also U17.9 (OUT1C); no longer U17.7 (RX2)
- net EN-2: now also U17.7 (RX2); no longer U17.9 (OUT1C)
- net EN-3: now also U17.5 (IN2); no longer U17.3 (LRCLK2)
- net EN-4: now also U17.3 (LRCLK2); no longer U17.5 (IN2)
- net EN-D: now also U19.5 (SDA_D4); no longer U19.6 (SCL_D5)
- net PH-1: now also U17.8 (TX2); no longer U17.6 (OUT1D)
- net PH-2: now also U17.6 (OUT1D); no longer U17.8 (TX2)
- net PH-3: now also U17.4 (BCLK2); no longer U17.2 (OUT2)
- net PH-4: now also U17.2 (OUT2); no longer U17.4 (BCLK2)
- net PH-D: now also U19.6 (SCL_D5); no longer U19.5 (SDA_D4)
- net SS: no longer names the net of J7.7 (Pin_7)
- net SS: no longer U17.10 (CS1)
- new net: JP2.1 (A), R20.1
- new net: JP1.1 (A), R19.1
- no-connect marks 14 -> 16
Other:
- moved on the sheet: D1, D2, R19, R20
