File: Schematic-PCB/Main-003-20241229/Main-003-20241229.kicad_pcb (KiCad board)
At the start: 4 copper layers, 112 x 112 mm, 96 parts, among them J1 Conn_PWR, J10 Conn_UI, J2 Conn_NeoPixel, J3 Conn_NeoPixel, J4 Conn_NeoPixel, J5 CamS3-6, J6 CamS3-4, J7 Pixy 2.1, J8 Conn_MD, J9 Conn_Dribbler, SW1 Main_RST, SW2 Cam_RST, SW3 Cam_RST, SW4 SW_DPDT_x2, U1 TSSP4038, U10 TSSP4038, U11 TSSP4038, U12 TSSP4038, U13 TSSP4038, U14 TSSP4038, U15 TSSP4038, U16 TSSP4038, U17 DEV-16771, U2 TSSP4038, U3 TSSP4038, U4 TSSP4038, U5 TSSP4038, U6 TSSP4038, U7 TSSP4038, U8 TSSP4038, U9 TSSP4038

Commit message: update: メイン基板のPCBを更新した
Parts:
- added JP1: Jumper_2_Small_Open, Jumper:SolderJumper-2_P1.3mm_Open_Pad1.0x1.5mm, B.Cu at (-15.0, 29.2)
- added JP2: Jumper_2_Small_Open, Jumper:SolderJumper-2_P1.3mm_Open_Pad1.0x1.5mm, B.Cu at (-15.0, 26.2)
- C1, C10, C11, C12, C13, C14, C15, C16, C2, C3, C4, C5, C6, C7, C8, C9, J1, J10, J9, R1, R10, R11, R12, R13, R14, R15, R16, R19, R2, R20, R21, R3, R4, R5, R6, R7, R8, R9: moved to B.Cu
- moved R4 234.2 mm to (-48.5, -9.66), turned to -101.25 degrees
- moved R3 233.8 mm to (-41.2, -27.5), turned to -123.75 degrees
- moved R2 227.2 mm to (-27.5, -41.2), turned to -146.25 degrees
- moved R5 225.6 mm to (-48.5, 9.66), turned to -78.75 degrees
- moved C4 223.3 mm to (-50.5, -10.0), turned to 78.75 degrees
- moved C3 222.1 mm to (-42.8, -28.6), turned to 56.25 degrees
- moved C5 218.1 mm to (-50.5, 10.0), turned to 101.25 degrees
- moved R6 215.5 mm to (-41.2, 27.5), turned to -56.25 degrees
- moved R1 214.7 mm to (-9.66, -48.5), turned to -168.75 degrees
- moved C2 214.5 mm to (-28.6, -42.8), turned to 33.75 degrees
- moved J1 211.1 mm to (-24.0, 19.0), turned to 123.75 degrees
- moved C6 206.9 mm to (-42.8, 28.6), turned to 123.75 degrees
- moved C1 201.1 mm to (-10.0, -50.5), turned to 11.25 degrees
- moved R7 200.6 mm to (-27.5, 41.2), turned to -33.75 degrees
- moved R20 199.3 mm to (-18.5, 26.2), turned to 180 degrees
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Connections:
- J7 pad 7: SS -> unconnected-(J7-Pin_7-Pad7)
- R19 pad 1: +5V -> Net-(JP1-A)
- R20 pad 1: +3.3V -> Net-(JP2-A)
- U17 pad 10: SS -> unconnected-(U17-CS1-Pad10)
- U17 pad 2: PH-3 -> PH-4
- U17 pad 3: EN-3 -> EN-4
- U17 pad 4: PH-4 -> PH-3
- U17 pad 5: EN-4 -> EN-3
- U17 pad 6: PH-1 -> PH-2
- U17 pad 7: EN-1 -> EN-2
- U17 pad 8: PH-2 -> PH-1
- U17 pad 9: EN-2 -> EN-1
- U19 pad 5: PH-D -> EN-D
- U19 pad 6: EN-D -> PH-D
Routing:
- net ball13: track 0.00 -> 103.9 mm, vias 0 -> 1
- net +5V: track 0.00 -> 86.0 mm, vias 0 -> 2
- net ball14: track 0.00 -> 82.6 mm, vias 0 -> 2
- net SW-TAC-2: track 0.00 -> 65.5 mm, vias 0 -> 1
- net ball03: track 0.00 -> 63.7 mm
- net SW-TAC-3: track 0.00 -> 63.2 mm, vias 0 -> 1
- net ball15: track 0.00 -> 62.5 mm
- net SW-TAC-4: track 0.00 -> 61.4 mm, vias 0 -> 1
- net ball02: track 0.00 -> 57.6 mm
- net ball04: track 0.00 -> 56.7 mm
- net ball10: track 0.00 -> 52.5 mm
- net SDA: track 0.00 -> 52.2 mm, vias 0 -> 1
- net ball01: track 0.00 -> 52.1 mm
- net SCL: track 0.00 -> 51.0 mm, vias 0 -> 2
- net ball16: track 0.00 -> 49.8 mm, vias 0 -> 1
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- added copper zone on F.Cu, net +3.3V
- added copper zone on B.Cu, net GND
Other:
- outline, holes or cut-outs redrawn
- copper layers 4 -> 2
- board text added: "+3.3V"
- board text added: "+5V"

Commit message: update: メイン基板のPCBを更新した
Parts:
- C19, C21, C23, C26, C27, C28, R17, R18: moved to B.Cu
- moved C22 208.0 mm to (-32.0, 10.0), turned to 90 degrees
- moved C25 204.7 mm to (-25.4, -5.08), turned to -90 degrees
- moved C28 202.4 mm to (0.00, -43.4)
- moved R22 195.3 mm to (0.00, -10.2)
- moved R23 195.3 mm to (0.00, -7.62)
- moved C21 189.6 mm to (-16.5, 19.1), turned to -90 degrees
- moved C23 188.8 mm to (-11.4, -1.91), turned to -90 degrees
- moved C19 174.7 mm to (-5.08, 27.9), turned to 90 degrees
- moved C24 172.9 mm to (15.2, -21.6), turned to -90 degrees
- moved C26 171.4 mm to (0.00, 30.5), turned to 180 degrees
- moved R18 166.7 mm to (16.5, 16.0), turned to 180 degrees
- moved C20 164.9 mm to (26.0, -15.9), turned to -90 degrees
- moved R17 164.4 mm to (16.5, 22.1), turned to 180 degrees
- moved C27 154.6 mm to (28.6, 0.00), turned to -90 degrees
- moved SW3 12.2 mm to (16.5, 16.0), turned to 180 degrees
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Routing:
- net ball11: track 2.00 -> 116.2 mm
- net ball12: track 2.00 -> 99.2 mm
- net Cam_EN: track 0.00 -> 49.7 mm
- net Cam_G0: track 0.00 -> 44.3 mm, vias 0 -> 3
- net Cam-RX: track 20.7 -> 54.5 mm, vias 0 -> 2
- net Cam-TX: track 21.1 -> 54.6 mm, vias 0 -> 1
- net Main_RST: track 23.4 -> 56.1 mm, vias 1 -> 0
- net GND: track 4.94 -> 26.2 mm
- net +3.3V: track 1.71 -> 17.8 mm, vias 1 -> 5
- net Net-(R21-Pad1): track 0.00 -> 13.7 mm
- net +5V: track 86.0 -> 98.2 mm
- net ball04: track 56.7 -> 57.9 mm
- net SCL: track 51.0 -> 52.2 mm, vias 2 -> 3
- net SDA: track 52.2 -> 53.4 mm, vias 1 -> 2
- net 3.3V: track 9.93 -> 10.4 mm
