File: Schematic-PCB/Line-004-20250115/Line-004-20250115.kicad_pcb (KiCad board)
At the start: 4 copper layers, 196 x 193.6 mm, 244 parts, among them J1 VIN, J2 Conn_MD, SW1 RESET, U47 LM393, U48 LM393, U49 LM393, U50 LM393, U51 LM393, U52 LM393, U53 LM393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

Commit message: update: ラインセンサ基板 ver.004 のフットプリントとPCBを編集した
Parts:
- removed C13, C16, C17, C18, C19: 100nF, Capacitor_SMD:C_0603_1608Metric
- removed C21, C22: 10uF, Capacitor_SMD:C_0805_2012Metric
- removed D47: LED01, LED_SMD:LED_0603_1608Metric
- removed JP10, JP7, JP8, JP9: Jumper_2_Small_Open, Jumper:SolderJumper-2_P1.3mm_Open_Pad1.0x1.5mm
- removed R79: 330, Resistor_SMD:R_0603_1608Metric
- removed R81, R84: 1K, Resistor_SMD:R_0603_1608Metric
- removed R86, R87: 100, Resistor_SMD:R_0603_1608Metric
- removed SW1: RESET, @2024TOINIOT2-Line:Tactile1
- removed U50: LM393, Package_SO:SOP-8_3.9x4.9mm_P1.27mm
- U62: footprint @2024TOINIOT2-Line:ATmega2560Pro Board -> @2024TOINIOT2-Line:ATmega2560Pro Board THT
- moved J1 2.75 mm to (1.25, 52.8)
- moved C20 0.91 mm to (-11.9, 49.5)
- turned U62 to 180 degrees
Routing:
- net Th2: track 354.8 -> 0.00 mm, vias 10 -> 0
- net Line-R: track 296.0 -> 0.00 mm, vias 6 -> 0
- net Line-B: track 203.9 -> 0.00 mm, vias 3 -> 0
- net 20: track 182.8 -> 0.00 mm, vias 2 -> 0
- net R: track 180.8 -> 0.00 mm, vias 2 -> 0
- net Line19: track 188.5 -> 9.27 mm, vias 4 -> 0
- net Line17: track 183.7 -> 9.27 mm, vias 2 -> 0
- net Line21: track 176.7 -> 8.83 mm, vias 1 -> 0
- net 21: track 164.2 -> 0.00 mm, vias 2 -> 0
- net 22: track 153.8 -> 0.00 mm, vias 2 -> 0
- net 18: track 146.4 -> 0.00 mm, vias 4 -> 0
- net Line15: track 166.1 -> 20.6 mm, vias 3 -> 0
- net 19: track 143.3 -> 0.00 mm, vias 4 -> 0
- net Line23: track 148.8 -> 8.83 mm, vias 1 -> 0
- net 23: track 137.1 -> 0.00 mm, vias 2 -> 0
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