File: Schematic-PCB/Line-004-20250115/Line-004-20250115.kicad_sch (KiCad schematic)
At the start: 221 parts, among them J1 VIN, J2 Conn_MD, SW1 RESET, U47 LM393, U48 LM393, U49 LM393, U50 LM393, U51 LM393, U52 LM393, U53 LM393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

Commit message: update: ラインセンサ基板 ver.004 のフットプリントとPCBを編集した
Parts:
- U62: footprint @2024TOINIOT2-Line:ATmega2560Pro Board -> @2024TOINIOT2-Line:ATmega2560Pro Board THT
Changed lines of the file:
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@@
 			)
 		)
-		(property "Footprint" "@2024TOINIOT2-Line:ATmega2560Pro Board"
+		(property "Footprint" "@2024TOINIOT2-Line:ATmega2560Pro Board THT"
 			(at 411.48 114.3 0)
 			(effects
